Commit message: refactor: setup harper monorepo and rename description package

File: harper_description/urdf/assemblies/harper_arm.urdf.xacro (robot description, xacro)
@@ -13,12 +13,12 @@
         <origin xyz="0.000000 0.000000 0.000000" rpy="0 0 0"/>
         <geometry>
-          <mesh filename="package://harper_arm_description/meshes/harper_arm/base_link.dae" scale="1 1 1"/>
-        </geometry>
-        <material name="ABS_Plastic"/>
-      </visual>
-      <collision>
-        <origin xyz="0.000000 0.000000 0.000000" rpy="0 0 0"/>
-        <geometry>
-          <mesh filename="package://harper_arm_description/meshes/harper_arm/base_link_collision.stl" scale="0.01 0.01 0.01"/>
+          <mesh filename="package://harper_description/meshes/harper_arm/base_link.dae" scale="1 1 1"/>
+        </geometry>
+        <material name="ABS_Plastic"/>
+      </visual>
+      <collision>
+        <origin xyz="0.000000 0.000000 0.000000" rpy="0 0 0"/>
+        <geometry>
+          <mesh filename="package://harper_description/meshes/harper_arm/base_link_collision.stl" scale="0.01 0.01 0.01"/>
         </geometry>
       </collision>
@@ -34,5 +34,5 @@
         <origin xyz="-0.127800 0.002450 -0.136700" rpy="0 0 0"/>
         <geometry>
-          <mesh filename="package://harper_arm_description/meshes/harper_arm/ubracket_link.dae" scale="1 1 1"/>
+          <mesh filename="package://harper_description/meshes/harper_arm/ubracket_link.dae" scale="1 1 1"/>
         </geometry>
         <material name="ABS_Plastic"/>
@@ -41,5 +41,5 @@
         <origin xyz="-0.127800 0.002450 -0.136700" rpy="0 0 0"/>
         <geometry>
-          <mesh filename="package://harper_arm_description/meshes/harper_arm/ubracket_link_collision.stl" scale="0.01 0.01 0.01"/>
+          <mesh filename="package://harper_description/meshes/harper_arm/ubracket_link_collision.stl" scale="0.01 0.01 0.01"/>
         </geometry>
       </collision>
@@ -55,5 +55,5 @@
         <origin xyz="-0.093300 0.039250 -0.136700" rpy="0 0 0"/>
         <geometry>
-          <mesh filename="package://harper_arm_description/meshes/harper_arm/abduction_link.dae" scale="1 1 1"/>
+          <mesh filename="package://harper_description/meshes/harper_arm/abduction_link.dae" scale="1 1 1"/>
         </geometry>
         <material name="ABS_Plastic"/>
@@ -62,5 +62,5 @@
         <origin xyz="-0.093300 0.039250 -0.136700" rpy="0 0 0"/>
         <geometry>
-          <mesh filename="package://harper_arm_description/meshes/harper_arm/abduction_link_collision.stl" scale="0.01 0.01 0.01"/>
+          <mesh filename="package://harper_description/meshes/harper_arm/abduction_link_collision.stl" scale="0.01 0.01 0.01"/>
         </geometry>
       </collision>
@@ -76,12 +76,12 @@
         <origin xyz="0.000000 0.000000 0.000000" rpy="0 0 0"/>
         <geometry>
-          <mesh filename="package://harper_arm_description/meshes/harper_arm/shoulder_rot_link.dae" scale="1 1 1"/>
-        </geometry>
-        <material name="ABS_Plastic"/>
-      </visual>
-      <collision>
-        <origin xyz="0.000000 0.000000 0.000000" rpy="0 0 0"/>
-        <geometry>
-          <mesh filename="package://harper_arm_description/meshes/harper_arm/shoulder_rot_link_collision.stl" scale="0.01 0.01 0.01"/>
+          <mesh filename="package://harper_description/meshes/harper_arm/shoulder_rot_link.dae" scale="1 1 1"/>
+        </geometry>
+        <material name="ABS_Plastic"/>
+      </visual>
+      <collision>
+        <origin xyz="0.000000 0.000000 0.000000" rpy="0 0 0"/>
+        <geometry>
+          <mesh filename="package://harper_description/meshes/harper_arm/shoulder_rot_link_collision.stl" scale="0.01 0.01 0.01"/>
         </geometry>
       </collision>
@@ -97,5 +97,5 @@
         <origin xyz="0.041000 0.152500 -0.012500" rpy="0 0 0"/>
         <geometry>
-          <mesh filename="package://harper_arm_description/meshes/harper_arm/elbow_forearm_link.dae" scale="1 1 1"/>
+          <mesh filename="package://harper_description/meshes/harper_arm/elbow_forearm_link.dae" scale="1 1 1"/>
         </geometry>
         <material name="ABS_Plastic"/>
@@ -104,5 +104,5 @@
         <origin xyz="0.041000 0.152500 -0.012500" rpy="0 0 0"/>
         <geometry>
-          <mesh filename="package://harper_arm_description/meshes/harper_arm/elbow_forearm_link_collision.stl" scale="0.01 0.01 0.01"/>
+          <mesh filename="package://harper_description/meshes/harper_arm/elbow_forearm_link_collision.stl" scale="0.01 0.01 0.01"/>
         </geometry>
       </collision>
@@ -118,5 +118,5 @@
         <origin xyz="-0.161425 -0.000000 0.000000" rpy="0 0 0"/>
         <geometry>
-          <mesh filename="package://harper_arm_description/meshes/harper_arm/forearm_front_link.dae" scale="1 1 1"/>
+          <mesh filename="package://harper_description/meshes/harper_arm/forearm_front_link.dae" scale="1 1 1"/>
         </geometry>
         <material name="ABS_Plastic"/>
@@ -125,5 +125,5 @@
         <origin xyz="-0.161425 -0.000000 0.000000" rpy="0 0 0"/>
         <geometry>
-          <mesh filename="package://harper_arm_description/meshes/harper_arm/forearm_front_link_collision.stl" scale="0.01 0.01 0.01"/>
+          <mesh filename="package://harper_description/meshes/harper_arm/forearm_front_link_collision.stl" scale="0.01 0.01 0.01"/>
         </geometry>
       </collision>

File: harper_description/urdf/harper_arm.urdf (robot description, URDF)
Before this commit: robot harper_arm, 6 links, 5 joints
Links:
- link abduction_link: geometry collision mesh filename=package://harper_description/meshes/harper_arm/abduction_li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 scale=0.01 0.01 0.01; visual mesh filename=package://harper_description/meshes/harper_arm/abduction_li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 scale=1 1 1
- link base_link: geometry collision mesh filename=package://harper_description/meshes/harper_arm/base_link_co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 scale=0.01 0.01 0.01; visual mesh filename=package://harper_description/meshes/harper_arm/base_link.dae scale=1 1 1
- link elbow_forearm_link: geometry collision mesh filename=package://harper_description/meshes/harper_arm/elbow_forear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 scale=0.01 0.01 0.01; visual mesh filename=package://harper_description/meshes/harper_arm/elbow_forear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 scale=1 1 1
- link forearm_front_link: geometry collision mesh filename=package://harper_description/meshes/harper_arm/forearm_fron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 scale=0.01 0.01 0.01; visual mesh filename=package://harper_description/meshes/harper_arm/forearm_fron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 scale=1 1 1
- link shoulder_rot_link: geometry collision mesh filename=package://harper_description/meshes/harper_arm/shoulder_rot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 scale=0.01 0.01 0.01; visual mesh filename=package://harper_description/meshes/harper_arm/shoulder_rot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 scale=1 1 1
- link ubracket_link: geometry collision mesh filename=package://harper_description/meshes/harper_arm/ubracket_lin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 scale=0.01 0.01 0.01; visual mesh filename=package://harper_description/meshes/harper_arm/ubracket_lin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 scale=1 1 1

File: harper_description/urdf/harper_arm.urdf.xacro (robot description, xacro)
@@ -6,5 +6,5 @@
   </material>
   <!-- Assembly includes -->
-  <xacro:include filename="$(find harper_arm_description)/urdf/assemblies/harper_arm.urdf.xacro"/>
+  <xacro:include filename="$(find harper_description)/urdf/assemblies/harper_arm.urdf.xacro"/>
   <!-- Instantiate assemblies -->
   <xacro:harper_arm prefix=""/>
