Commit message: chore(sync): add dual-arm control/motion stack and init docs site page

File: harper_description/urdf/assemblies/left_arm.urdf.xacro (robot description, xacro)
@@ -606,4 +606,5 @@
       <axis xyz="-0.999727 -0.022418 -0.006632"/>
       <limit lower="-0.785398" upper="0.698132" effort="100.0" velocity="1.00"/>
+      <mimic joint="${prefix}left_thb_mip_joint" multiplier="1.0" offset="0.0"/>
     </joint>
     <joint name="${prefix}left_ind_pip_joint" type="revolute">
@@ -613,4 +614,5 @@
       <axis xyz="-1.000000 -0.000495 -0.000829"/>
       <limit lower="-0.698132" upper="1.047198" effort="100.0" velocity="1.00"/>
+      <mimic joint="${prefix}left_ind_mip_joint" multiplier="1.0" offset="0.0"/>
     </joint>
     <joint name="${prefix}left_mid_pip_joint" type="revolute">
@@ -620,4 +622,5 @@
       <axis xyz="-1.000000 -0.000273 -0.000220"/>
       <limit lower="-0.959931" upper="0.610865" effort="100.0" velocity="1.00"/>
+      <mimic joint="${prefix}left_mid_mip_joint" multiplier="1.0" offset="0.0"/>
     </joint>
     <joint name="${prefix}left_rng_pip_joint" type="revolute">
@@ -627,4 +630,5 @@
       <axis xyz="-0.998865 -0.041252 -0.023803"/>
       <limit lower="-0.785398" upper="0.610865" effort="100.0" velocity="1.00"/>
+      <mimic joint="${prefix}left_rng_mip_joint" multiplier="1.0" offset="0.0"/>
     </joint>
     <joint name="${prefix}left_pnk_pip_joint" type="revolute">
@@ -634,4 +638,5 @@
       <axis xyz="-0.999417 -0.029916 -0.016475"/>
       <limit lower="-0.872665" upper="0.698132" effort="100.0" velocity="1.00"/>
+      <mimic joint="${prefix}left_pnk_mip_joint" multiplier="1.0" offset="0.0"/>
     </joint>
     <joint name="${prefix}left_ind_dip_joint" type="revolute">
@@ -641,4 +646,5 @@
       <axis xyz="-1.000000 0.000497 -0.000831"/>
       <limit lower="-0.872665" upper="0.698132" effort="100.0" velocity="1.00"/>
+      <mimic joint="${prefix}left_ind_mip_joint" multiplier="1.0" offset="0.0"/>
     </joint>
     <joint name="${prefix}left_mid_dip_joint" type="revolute">
@@ -648,4 +654,5 @@
       <axis xyz="-1.000000 0.000497 -0.000831"/>
       <limit lower="-0.785398" upper="0.436332" effort="100.0" velocity="1.00"/>
+      <mimic joint="${prefix}left_mid_mip_joint" multiplier="1.0" offset="0.0"/>
     </joint>
     <joint name="${prefix}left_rng_dip_joint" type="revolute">
@@ -655,4 +662,5 @@
       <axis xyz="-0.999953 -0.008229 -0.005153"/>
       <limit lower="-0.959931" upper="0.523599" effort="100.0" velocity="1.00"/>
+      <mimic joint="${prefix}left_rng_mip_joint" multiplier="1.0" offset="0.0"/>
     </joint>
     <joint name="${prefix}left_pnk_dip_joint" type="revolute">
@@ -662,193 +670,7 @@
       <axis xyz="-1.000000 -0.000000 0.000001"/>
       <limit lower="-0.436332" upper="0.785398" effort="100.0" velocity="1.00"/>
-    </joint>
-    <!-- ROS 2 control: generated generic system -->
-    <ros2_control name="${prefix}left_arm_system" type="system">
-      <hardware>
-        <plugin>mock_components/GenericSystem</plugin>
-        <param name="cmd_topic">sim/left_arm_system/cmd</param>
-        <param name="state_topic">sim/left_arm_system/state</param>
-      </hardware>
-      <joint name="${prefix}left_elb_fex_joint">
-        <command_interface name="position"/>
-        <command_interface name="velocity"/>
-        <state_interface name="position">
-          <param name="initial_value">0.0</param>
-        </state_interface>
-        <state_interface name="velocity"/>
-        <state_interface name="effort"/>
-      </joint>
-      <joint name="${prefix}left_fam_rot_joint">
-        <command_interface name="position"/>
-        <command_interface name="velocity"/>
-        <state_interface name="position">
-          <param name="initial_value">0.0</param>
-        </state_interface>
-        <state_interface name="velocity"/>
-        <state_interface name="effort"/>
-      </joint>
-      <joint name="${prefix}left_ind_dip_joint">
-        <command_interface name="position"/>
-        <command_interface name="velocity"/>
-        <state_interface name="position">
-          <param name="initial_value">0.0</param>
-        </state_interface>
-        <state_interface name="velocity"/>
-        <state_interface name="effort"/>
-      </joint>
-      <joint name="${prefix}left_ind_mip_joint">
-        <command_interface name="position"/>
-        <command_interface name="velocity"/>
-        <state_interface name="position">
-          <param name="initial_value">0.0</param>
-        </state_interface>
-        <state_interface name="velocity"/>
-        <state_interface name="effort"/>
-      </joint>
-      <joint name="${prefix}left_ind_pip_joint">
-        <command_interface name="position"/>
-        <command_interface name="velocity"/>
-        <state_interface name="position">
-          <param name="initial_value">0.0</param>
-        </state_interface>
-        <state_interface name="velocity"/>
-        <state_interface name="effort"/>
-      </joint>
-      <joint name="${prefix}left_mid_dip_joint">
-        <command_interface name="position"/>
-        <command_interface name="velocity"/>
-        <state_interface name="position">
-          <param name="initial_value">0.0</param>
-        </state_interface>
-        <state_interface name="velocity"/>
-        <state_interface name="effort"/>
-      </joint>
-      <joint name="${prefix}left_mid_mip_joint">
-        <command_interface name="position"/>
-        <command_interface name="velocity"/>
-        <state_interface name="position">
-          <param name="initial_value">0.0</param>
-        </state_interface>
-        <state_interface name="velocity"/>
-        <state_interface name="effort"/>
-      </joint>
-      <joint name="${prefix}left_mid_pip_joint">
-        <command_interface name="position"/>
-        <command_interface name="velocity"/>
-        <state_interface name="position">
-          <param name="initial_value">0.0</param>
-        </state_interface>
-        <state_interface name="velocity"/>
-        <state_interface name="effort"/>
-      </joint>
-      <joint name="${prefix}left_pnk_dip_joint">
-        <command_interface name="position"/>
-        <command_interface name="velocity"/>
-        <state_interface name="position">
-          <param name="initial_value">0.0</param>
-        </state_interface>
-        <state_interface name="velocity"/>
-        <state_interface name="effort"/>
-      </joint>
-      <joint name="${prefix}left_pnk_mip_joint">
-        <command_interface name="position"/>
-        <command_interface name="velocity"/>
-        <state_interface name="position">
-          <param name="initial_value">0.0</param>
-        </state_interface>
-        <state_interface name="velocity"/>
-        <state_interface name="effort"/>
-      </joint>
-      <joint name="${prefix}left_pnk_pip_joint">
-        <command_interface name="position"/>
-        <command_interface name="velocity"/>
-        <state_interface name="position">
-          <param name="initial_value">0.0</param>
-        </state_interface>
-        <state_interface name="velocity"/>
-        <state_interface name="effort"/>
-      </joint>
-      <joint name="${prefix}left_rng_dip_joint">
-        <command_interface name="position"/>
-        <command_interface name="velocity"/>
-        <state_interface name="position">
-          <param name="initial_value">0.0</param>
-        </state_interface>
-        <state_interface name="velocity"/>
-        <state_interface name="effort"/>
-      </joint>
-      <joint name="${prefix}left_rng_mip_joint">
-        <command_interface name="position"/>
-        <command_interface name="velocity"/>
-        <state_interface name="position">
-          <param name="initial_value">0.0</param>
-        </state_interface>
-        <state_interface name="velocity"/>
-        <state_interface name="effort"/>
-      </joint>
-      <joint name="${prefix}left_rng_pip_joint">
-        <command_interface name="position"/>
-        <command_interface name="velocity"/>
-        <state_interface name="position">
-          <param name="initial_value">0.0</param>
-        </state_interface>
-        <state_interface name="velocity"/>
-        <state_interface name="effort"/>
-      </joint>
-      <joint name="${prefix}left_shd_aad_joint">
-        <command_interface name="position"/>
-        <command_interface name="velocity"/>
-        <state_interface name="position">
-          <param name="initial_value">0.0</param>
-        </state_interface>
-        <state_interface name="velocity"/>
-        <state_interface name="effort"/>
-      </joint>
-      <joint name="${prefix}left_shd_fex_joint">
-        <command_interface name="position"/>
-        <command_interface name="velocity"/>
-        <state_interface name="position">
-          <param name="initial_value">0.0</param>
-        </state_interface>
-        <state_interface name="velocity"/>
-        <state_interface name="effort"/>
-      </joint>
-      <joint name="${prefix}left_shd_rot_joint">
-        <command_interface name="position"/>
-        <command_interface name="velocity"/>
-        <state_interface name="position">
-          <param name="initial_value">0.0</param>
-        </state_interface>
-        <state_interface name="velocity"/>
-        <state_interface name="effort"/>
-      </joint>
-      <joint name="${prefix}left_thb_ip_joint">
-        <command_interface name="position"/>
-        <command_interface name="velocity"/>
-        <state_interface name="position">
-          <param name="initial_value">0.0</param>
-        </state_interface>
-        <state_interface name="velocity"/>
-        <state_interface name="effort"/>
-      </joint>
-      <joint name="${prefix}left_thb_mip_joint">
-        <command_interface name="position"/>
-        <command_interface name="velocity"/>
-        <state_interface name="position">
-          <param name="initial_value">0.0</param>
-        </state_interface>
-        <state_interface name="velocity"/>
-        <state_interface name="effort"/>
-      </joint>
-      <joint name="${prefix}left_wrs_fex_joint">
-        <command_interface name="position"/>
-        <command_interface name="velocity"/>
-        <state_interface name="position">
-          <param name="initial_value">0.0</param>
-        </state_interface>
-        <state_interface name="velocity"/>
-        <state_interface name="effort"/>
-      </joint>
-    </ros2_control>
+      <mimic joint="${prefix}left_pnk_mip_joint" multiplier="1.0" offset="0.0"/>
+    </joint>
+    <!-- ros2_control lives in urdf/harper_ros2_control.xacro (single dual-arm system). -->
   </xacro:macro>
 </robot>

File: harper_description/urdf/assemblies/right_arm.urdf.xacro (robot description, xacro)
@@ -553,5 +553,5 @@
       <limit lower="-2.356194" upper="2.356194" effort="100.0" velocity="1.00"/>
     </joint>
-    <joint name="${prefix}right_wrist_fex_joint" type="revolute">
+    <joint name="${prefix}right_wrs_fex_joint" type="revolute">
       <parent link="${prefix}right_wrs_upp_link"/>
       <child link="${prefix}right_wrs_low_link"/>
@@ -606,4 +606,5 @@
       <axis xyz="1.000000 0.000244 0.000407"/>
       <limit lower="-1.047198" upper="0.349066" effort="100.0" velocity="1.00"/>
+      <mimic joint="${prefix}right_thb_mip_joint" multiplier="1.0" offset="0.0"/>
     </joint>
     <joint name="${prefix}right_ind_pip_joint" type="revolute">
@@ -613,4 +614,5 @@
       <axis xyz="-1.000000 -0.000495 0.000829"/>
       <limit lower="-0.872665" upper="0.523599" effort="100.0" velocity="1.00"/>
+      <mimic joint="${prefix}right_ind_mip_joint" multiplier="1.0" offset="0.0"/>
     </joint>
     <joint name="${prefix}right_mid_pip_joint" type="revolute">
@@ -620,4 +622,5 @@
       <axis xyz="-1.000000 -0.000273 0.000220"/>
       <limit lower="-0.959931" upper="0.523599" effort="100.0" velocity="1.00"/>
+      <mimic joint="${prefix}right_mid_mip_joint" multiplier="1.0" offset="0.0"/>
     </joint>
     <joint name="${prefix}right_rng_pip_joint" type="revolute">
@@ -627,4 +630,5 @@
       <axis xyz="1.000000 -0.000000 0.000000"/>
       <limit lower="2.094395" upper="3.316126" effort="100.0" velocity="1.00"/>
+      <mimic joint="${prefix}right_rng_mip_joint" multiplier="1.0" offset="0.0"/>
     </joint>
     <joint name="${prefix}right_pnk_pip_joint" type="revolute">
@@ -634,4 +638,5 @@
       <axis xyz="-0.999913 0.011060 -0.007127"/>
       <limit lower="-0.698132" upper="0.872665" effort="100.0" velocity="1.00"/>
+      <mimic joint="${prefix}right_pnk_mip_joint" multiplier="1.0" offset="0.0"/>
     </joint>
     <joint name="${prefix}right_ind_dip_joint" type="revolute">
@@ -641,4 +646,5 @@
       <axis xyz="1.000000 -0.000497 -0.000831"/>
       <limit lower="-0.785398" upper="0.523599" effort="100.0" velocity="1.00"/>
+      <mimic joint="${prefix}right_ind_mip_joint" multiplier="1.0" offset="0.0"/>
     </joint>
     <joint name="${prefix}right_mid_dip_joint" type="revolute">
@@ -648,4 +654,5 @@
       <axis xyz="0.999832 -0.016197 0.008554"/>
       <limit lower="-0.872665" upper="0.436332" effort="100.0" velocity="1.00"/>
+      <mimic joint="${prefix}right_mid_mip_joint" multiplier="1.0" offset="0.0"/>
     </joint>
     <joint name="${prefix}right_rng_dip_joint" type="revolute">
@@ -655,4 +662,5 @@
       <axis xyz="-1.000000 0.000265 0.000482"/>
       <limit lower="-0.523599" upper="0.872665" effort="100.0" velocity="1.00"/>
+      <mimic joint="${prefix}right_rng_mip_joint" multiplier="1.0" offset="0.0"/>
     </joint>
     <joint name="${prefix}right_pnk_dip_joint" type="revolute">
@@ -662,193 +670,7 @@
       <axis xyz="-0.999632 -0.022709 0.014809"/>
       <limit lower="-0.436332" upper="0.959931" effort="100.0" velocity="1.00"/>
-    </joint>
-    <!-- ROS 2 control: generated generic system -->
-    <ros2_control name="${prefix}right_arm_system" type="system">
-      <hardware>
-        <plugin>mock_components/GenericSystem</plugin>
-        <param name="cmd_topic">sim/right_arm_system/cmd</param>
-        <param name="state_topic">sim/right_arm_system/state</param>
-      </hardware>
-      <joint name="${prefix}right_elb_fex_joint">
-        <command_interface name="position"/>
-        <command_interface name="velocity"/>
-        <state_interface name="position">
-          <param name="initial_value">0.0</param>
-        </state_interface>
-        <state_interface name="velocity"/>
-        <state_interface name="effort"/>
-      </joint>
-      <joint name="${prefix}right_fam_rot_joint">
-        <command_interface name="position"/>
-        <command_interface name="velocity"/>
-        <state_interface name="position">
-          <param name="initial_value">0.0</param>
-        </state_interface>
-        <state_interface name="velocity"/>
-        <state_interface name="effort"/>
-      </joint>
-      <joint name="${prefix}right_ind_dip_joint">
-        <command_interface name="position"/>
-        <command_interface name="velocity"/>
-        <state_interface name="position">
-          <param name="initial_value">0.0</param>
-        </state_interface>
-        <state_interface name="velocity"/>
-        <state_interface name="effort"/>
-      </joint>
-      <joint name="${prefix}right_ind_mip_joint">
-        <command_interface name="position"/>
-        <command_interface name="velocity"/>
-        <state_interface name="position">
-          <param name="initial_value">0.0</param>
-        </state_interface>
-        <state_interface name="velocity"/>
-        <state_interface name="effort"/>
-      </joint>
-      <joint name="${prefix}right_ind_pip_joint">
-        <command_interface name="position"/>
-        <command_interface name="velocity"/>
-        <state_interface name="position">
-          <param name="initial_value">0.0</param>
-        </state_interface>
-        <state_interface name="velocity"/>
-        <state_interface name="effort"/>
-      </joint>
-      <joint name="${prefix}right_mid_dip_joint">
-        <command_interface name="position"/>
-        <command_interface name="velocity"/>
-        <state_interface name="position">
-          <param name="initial_value">0.0</param>
-        </state_interface>
-        <state_interface name="velocity"/>
-        <state_interface name="effort"/>
-      </joint>
-      <joint name="${prefix}right_mid_mip_joint">
-        <command_interface name="position"/>
-        <command_interface name="velocity"/>
-        <state_interface name="position">
-          <param name="initial_value">0.0</param>
-        </state_interface>
-        <state_interface name="velocity"/>
-        <state_interface name="effort"/>
-      </joint>
-      <joint name="${prefix}right_mid_pip_joint">
-        <command_interface name="position"/>
-        <command_interface name="velocity"/>
-        <state_interface name="position">
-          <param name="initial_value">0.0</param>
-        </state_interface>
-        <state_interface name="velocity"/>
-        <state_interface name="effort"/>
-      </joint>
-      <joint name="${prefix}right_pnk_dip_joint">
-        <command_interface name="position"/>
-        <command_interface name="velocity"/>
-        <state_interface name="position">
-          <param name="initial_value">0.0</param>
-        </state_interface>
-        <state_interface name="velocity"/>
-        <state_interface name="effort"/>
-      </joint>
-      <joint name="${prefix}right_pnk_mip_joint">
-        <command_interface name="position"/>
-        <command_interface name="velocity"/>
-        <state_interface name="position">
-          <param name="initial_value">0.0</param>
-        </state_interface>
-        <state_interface name="velocity"/>
-        <state_interface name="effort"/>
-      </joint>
-      <joint name="${prefix}right_pnk_pip_joint">
-        <command_interface name="position"/>
-        <command_interface name="velocity"/>
-        <state_interface name="position">
-          <param name="initial_value">0.0</param>
-        </state_interface>
-        <state_interface name="velocity"/>
-        <state_interface name="effort"/>
-      </joint>
-      <joint name="${prefix}right_rng_dip_joint">
-        <command_interface name="position"/>
-        <command_interface name="velocity"/>
-        <state_interface name="position">
-          <param name="initial_value">0.0</param>
-        </state_interface>
-        <state_interface name="velocity"/>
-        <state_interface name="effort"/>
-      </joint>
-      <joint name="${prefix}right_rng_mip_joint">
-        <command_interface name="position"/>
-        <command_interface name="velocity"/>
-        <state_interface name="position">
-          <param name="initial_value">0.0</param>
-        </state_interface>
-        <state_interface name="velocity"/>
-        <state_interface name="effort"/>
-      </joint>
-      <joint name="${prefix}right_rng_pip_joint">
-        <command_interface name="position"/>
-        <command_interface name="velocity"/>
-        <state_interface name="position">
-          <param name="initial_value">0.0</param>
-        </state_interface>
-        <state_interface name="velocity"/>
-        <state_interface name="effort"/>
-      </joint>
-      <joint name="${prefix}right_shd_aad_joint">
-        <command_interface name="position"/>
-        <command_interface name="velocity"/>
-        <state_interface name="position">
-          <param name="initial_value">0.0</param>
-        </state_interface>
-        <state_interface name="velocity"/>
-        <state_interface name="effort"/>
-      </joint>
-      <joint name="${prefix}right_shd_fex_joint">
-        <command_interface name="position"/>
-        <command_interface name="velocity"/>
-        <state_interface name="position">
-          <param name="initial_value">0.0</param>
-        </state_interface>
-        <state_interface name="velocity"/>
-        <state_interface name="effort"/>
-      </joint>
-      <joint name="${prefix}right_shd_rot_joint">
-        <command_interface name="position"/>
-        <command_interface name="velocity"/>
-        <state_interface name="position">
-          <param name="initial_value">0.0</param>
-        </state_interface>
-        <state_interface name="velocity"/>
-        <state_interface name="effort"/>
-      </joint>
-      <joint name="${prefix}right_thb_ip_joint">
-        <command_interface name="position"/>
-        <command_interface name="velocity"/>
-        <state_interface name="position">
-          <param name="initial_value">0.0</param>
-        </state_interface>
-        <state_interface name="velocity"/>
-        <state_interface name="effort"/>
-      </joint>
-      <joint name="${prefix}right_thb_mip_joint">
-        <command_interface name="position"/>
-        <command_interface name="velocity"/>
-        <state_interface name="position">
-          <param name="initial_value">0.0</param>
-        </state_interface>
-        <state_interface name="velocity"/>
-        <state_interface name="effort"/>
-      </joint>
-      <joint name="${prefix}right_wrist_fex_joint">
-        <command_interface name="position"/>
-        <command_interface name="velocity"/>
-        <state_interface name="position">
-          <param name="initial_value">0.0</param>
-        </state_interface>
-        <state_interface name="velocity"/>
-        <state_interface name="effort"/>
-      </joint>
-    </ros2_control>
+      <mimic joint="${prefix}right_pnk_mip_joint" multiplier="1.0" offset="0.0"/>
+    </joint>
+    <!-- ros2_control lives in urdf/harper_ros2_control.xacro (single dual-arm system). -->
   </xacro:macro>
 </robot>

File: harper_description/urdf/harper.urdf (robot description, URDF)
Before this commit: robot harper, 50 links, 49 joints
Joints:
- removed joint right_wrist_fex_joint
- added joint right_wrs_fex_joint: type revolute, parent right_wrs_upp_link, child right_wrs_low_link, origin xyz=-0.019216 0.049400 0.000018 rpy=-1.570796 -0.000000 -0.000000, axis -1.000000 0.000000 -0.000000, limit lower=-1.221730 upper=1.570796 effort=100.0 velocity=1.00
